Commit message: add my_robot 2 wheels

File: my_robot/urdf/my_robot.xacro (robot description, xacro)
@@ -2,9 +2,4 @@
 <robot name="my_robot" xmlns:xacro="http://www.ros.org/wiki/xacro">
     <link name="robot_footprint"></link>
-    <joint name="robot_footprint_joint" type="fixed">
-        <origin xyz="0 0 0" rpy="0 0 0" />
-        <parent link="robot_footprint" />
-        <child link="chassis" />
-    </joint>
     <link name='chassis'>
         <pose>0 0 0.1 0 0 0</pose>
@@ -15,8 +10,7 @@
                 ixx="0.1" ixy="0" ixz="0"
                 iyy="0.1" iyz="0"
-                izz="0.1"
-            />
+                izz="0.1" />
         </inertial>
-        <collision name='collision'>
+        <collision name='chassis_collision'>
             <origin xyz="0 0 0" rpy=" 0 0 0" />
             <geometry>
@@ -43,5 +37,5 @@
         </visual>
         <collision name='front_caster_collision'>
-            <origin xyz="0.15 0 -0.05" rpy=" 0 0 0" />
+            <origin xyz="0.15 0 -0.05" rpy="0 0 0" />
             <geometry>
                 <sphere radius="0.0499" />
@@ -49,5 +43,5 @@
         </collision>
         <visual name='front_caster_visual'>
-            <origin xyz="0.15 0 -0.05" rpy=" 0 0 0" />
+            <origin xyz="0.15 0 -0.05" rpy="0 0 0" />
             <geometry>
                 <sphere radius="0.05" />
@@ -55,3 +49,68 @@
         </visual>
     </link>
+    <joint name="robot_footprint_joint" type="fixed">
+        <origin xyz="0 0 0" rpy="0 0 0" />
+        <parent link="robot_footprint" />
+        <child link="chassis" />
+    </joint>
+    <link name='left_wheel'>
+        <inertial>
+            <mass value="5.0" />
+            <origin xyz="0.0 0 0" rpy="0 0 0" />
+            <inertia
+                ixx="0.1" ixy="0" ixz="0"
+                iyy="0.1" iyz="0"
+                izz="0.1" />
+        </inertial>
+        <visual name='left_wheel_visual'>
+            <origin xyz="0 0 0" rpy="0 1.5707 1.5707" />
+            <geometry>
+                <cylinder radius="0.1" length="0.05" />
+            </geometry>
+        </visual>
+        <collision name='left_wheel_collision'>
+            <origin xyz="0 0 0" rpy="0 1.5707 1.5707" />
+            <geometry>
+                <cylinder radius="0.099" length="0.0499" />
+            </geometry>
+        </collision>
+    </link>
+    <joint type="continuous" name="left_wheel_hinge">
+        <origin xyz="0 0.15 0" rpy="0 0 0" />
+        <child link="left_wheel" />
+        <parent link="chassis" />
+        <axis xyz="0 1 0" rpy="0 0 0" />
+        <limit effort="10000" velocity="1000" />
+        <dynamics damping="1.0" friction="1.0" />
+    </joint>
+    <link name='right_wheel'>
+        <inertial>
+            <mass value="5.0" />
+            <origin xyz="0.0 0 0" rpy=" 0 0 0" />
+            <inertia
+                ixx="0.1" ixy="0" ixz="0"
+                iyy="0.1" iyz="0"
+                izz="0.1" />
+        </inertial>
+        <visual name='right_wheel_visual'>
+            <origin xyz="0 0 0" rpy="0 1.5707 1.5707" />
+            <geometry>
+                <cylinder radius="0.1" length="0.05" />
+            </geometry>
+        </visual>
+        <collision name='right_wheel_collision'>
+            <origin xyz="0 0 0" rpy="0 1.5707 1.5707" />
+            <geometry>
+                <cylinder radius="0.099" length="0.0499" />
+            </geometry>
+        </collision>
+    </link>
+    <joint type="continuous" name="right_wheel_hinge">
+        <origin xyz="0 0.15 0" rpy="0 0 0" />
+        <child link="right_wheel" />
+        <parent link="chassis" />
+        <axis xyz="0 1 0" rpy="0 0 0" />
+        <limit effort="10000" velocity="1000" />
+        <dynamics damping="1.0" friction="1.0" />
+    </joint>
 </robot>

Commit message: .

File: my_robot/urdf/my_robot.xacro (robot description, xacro)
@@ -107,5 +107,5 @@
     </link>
     <joint type="continuous" name="right_wheel_hinge">
-        <origin xyz="0 0.15 0" rpy="0 0 0" />
+        <origin xyz="0 -0.15 0" rpy="0 0 0" />
         <child link="right_wheel" />
         <parent link="chassis" />

Commit message: create camera link

File: my_robot/urdf/my_robot.xacro (robot description, xacro)
@@ -114,3 +114,32 @@
         <dynamics damping="1.0" friction="1.0" />
     </joint>
+    <!-- Camera link -->
+    <link name="camera">
+        <origin xyz="0 0 0" rpy="0 0 0" />
+        <inertial>
+            <mass value="0.1" />
+            <origin xyz="0 0 0" rpy="0 0 0" />
+            <inertia ixx="1e-6" ixy="0" ixz="0" iyy="1e-6" iyz="0" izz="1e-6" />
+        </inertial>
+        <visual>
+            <origin xyz="0 0 0" rpy="0 0 0" />
+            <geometry>
+                <box size="0.05 0.05 0.05" />
+            </geometry>
+            <material name="grey" />
+        </visual>
+        <collision>
+            <origin xyz="0 0 0" rpy="0 0 0" />
+            <geometry>
+                <box size="0.05 0.05 0.05" />
+            </geometry>
+        </collision>
+    </link>
+    <!-- Camera joint -->
+    <joint name="camera_joint" type="fixed">
+        <parent link="chassis" />
+        <child link="camera" />
+        <origin xyz="0.2 0 0" rpy="0 0 0" />
+        <axis xyz="0 1 0" />
+    </joint>
 </robot>

Commit message: add lidar to my_robot

File: my_robot/urdf/my_robot.xacro (robot description, xacro)
@@ -143,3 +143,31 @@
         <axis xyz="0 1 0" />
     </joint>
+    <!-- Hokuyo LiDAR link -->
+    <link name="hokuyo">
+        <origin xyz="0 0 0" rpy="0 0 0" />
+        <inertial>
+            <mass value="1e-5" />
+            <origin xyz="0 0 0" rpy="0 0 0" />
+            <inertia ixx="1e-6" ixy="0" ixz="0" iyy="1e-6" iyz="0" izz="1e-6" />
+        </inertial>
+        <visual>
+            <origin xyz="0 0 0" rpy="0 0 0" />
+            <geometry>
+                <mesh filename="package://my_robot/meshes/hokuyo.dae" />
+            </geometry>
+        </visual>
+        <collision>
+            <origin xyz="0 0 0" rpy="0 0 0" />
+            <geometry>
+                <box size="0.1 0.1 0.1" />
+            </geometry>
+        </collision>
+    </link>
+    <!-- Hokuyo LiDAR joint -->
+    <joint name="hokuyo_joint" type="fixed">
+        <parent link="chassis" />
+        <child link="hokuyo" />
+        <origin xyz="0.15 0 0.1" rpy="0 0 0" />
+        <axis xyz="0 1 0" />
+    </joint>
 </robot>

Commit message: set material for my_robot

File: my_robot/urdf/my_robot.xacro (robot description, xacro)
@@ -49,4 +49,7 @@
         </visual>
     </link>
+    <gazebo reference="chassis">
+        <material>Gazebo/Wood</material>
+    </gazebo>
     <joint name="robot_footprint_joint" type="fixed">
         <origin xyz="0 0 0" rpy="0 0 0" />
@@ -76,4 +79,7 @@
         </collision>
     </link>
+    <gazebo reference="left_wheel">
+        <material>Gazebo/Gold</material>
+    </gazebo>
     <joint type="continuous" name="left_wheel_hinge">
         <origin xyz="0 0.15 0" rpy="0 0 0" />

Commit message: .

File: my_robot/urdf/my_robot.xacro (robot description, xacro)
@@ -2,4 +2,17 @@
 <robot name="my_robot" xmlns:xacro="http://www.ros.org/wiki/xacro">
     <link name="robot_footprint"></link>
+    <!-- Model materials -->
+    <gazebo reference="chassis">
+        <material>Gazebo/WoodPallet</material>
+    </gazebo>
+    <gazebo reference="left_wheel">
+        <material>Gazebo/GreyTransparent</material>
+    </gazebo>
+    <gazebo reference="right_wheel">
+        <material>Gazebo/GreyTransparent</material>
+    </gazebo>
+    <gazebo reference="hokuyo">
+        <material>Gazebo/GreenGlow</material>
+    </gazebo>
     <link name='chassis'>
         <pose>0 0 0.1 0 0 0</pose>
@@ -49,7 +62,4 @@
         </visual>
     </link>
-    <gazebo reference="chassis">
-        <material>Gazebo/Wood</material>
-    </gazebo>
     <joint name="robot_footprint_joint" type="fixed">
         <origin xyz="0 0 0" rpy="0 0 0" />
@@ -79,7 +89,4 @@
         </collision>
     </link>
-    <gazebo reference="left_wheel">
-        <material>Gazebo/Gold</material>
-    </gazebo>
     <joint type="continuous" name="left_wheel_hinge">
         <origin xyz="0 0.15 0" rpy="0 0 0" />

Commit message: .

File: my_robot/urdf/my_robot.xacro (robot description, xacro)
@@ -4,5 +4,5 @@
     <!-- Model materials -->
     <gazebo reference="chassis">
-        <material>Gazebo/WoodPallet</material>
+        <material>Gazebo/WoodFloor</material>
     </gazebo>
     <gazebo reference="left_wheel">
@@ -12,6 +12,6 @@
         <material>Gazebo/GreyTransparent</material>
     </gazebo>
-    <gazebo reference="hokuyo">
-        <material>Gazebo/GreenGlow</material>
+    <gazebo reference="camera">
+        <material>Gazebo/LightBlueLaser</material>
     </gazebo>
     <link name='chassis'>

Commit message: .

File: my_robot/urdf/my_robot.xacro (robot description, xacro)
@@ -7,11 +7,11 @@
     </gazebo>
     <gazebo reference="left_wheel">
-        <material>Gazebo/GreyTransparent</material>
+        <material>Gazebo/PaintedWall</material>
     </gazebo>
     <gazebo reference="right_wheel">
-        <material>Gazebo/GreyTransparent</material>
+        <material>Gazebo/PaintedWall</material>
     </gazebo>
     <gazebo reference="camera">
-        <material>Gazebo/LightBlueLaser</material>
+        <material>Gazebo/Green</material>
     </gazebo>
     <link name='chassis'>

Commit message: .

File: my_robot/urdf/my_robot.xacro (robot description, xacro)
@@ -4,11 +4,11 @@
     <!-- Model materials -->
     <gazebo reference="chassis">
-        <material>Gazebo/WoodFloor</material>
+        <material>Gazebo/Wood</material>
     </gazebo>
     <gazebo reference="left_wheel">
-        <material>Gazebo/PaintedWall</material>
+        <material>Gazebo/PioneerBody</material>
     </gazebo>
     <gazebo reference="right_wheel">
-        <material>Gazebo/PaintedWall</material>
+        <material>Gazebo/PioneerBody</material>
     </gazebo>
     <gazebo reference="camera">

Commit message: .

File: my_robot/urdf/my_robot.xacro (robot description, xacro)
@@ -7,8 +7,8 @@
     </gazebo>
     <gazebo reference="left_wheel">
-        <material>Gazebo/PioneerBody</material>
+        <material>Gazebo/CloudySky</material>
     </gazebo>
     <gazebo reference="right_wheel">
-        <material>Gazebo/PioneerBody</material>
+        <material>Gazebo/CloudySky</material>
     </gazebo>
     <gazebo reference="camera">

Commit message: .

File: my_robot/urdf/my_robot.xacro (robot description, xacro)
@@ -7,11 +7,11 @@
     </gazebo>
     <gazebo reference="left_wheel">
-        <material>Gazebo/CloudySky</material>
+        <material>Gazebo/BlackTransparent</material>
     </gazebo>
     <gazebo reference="right_wheel">
-        <material>Gazebo/CloudySky</material>
+        <material>Gazebo/BlackTransparent</material>
     </gazebo>
     <gazebo reference="camera">
-        <material>Gazebo/Green</material>
+        <material>Gazebo/GreenTransparentOverlay</material>
     </gazebo>
     <link name='chassis'>

Commit message: .

File: my_robot/urdf/my_robot.xacro (robot description, xacro)
@@ -7,8 +7,8 @@
     </gazebo>
     <gazebo reference="left_wheel">
-        <material>Gazebo/BlackTransparent</material>
+        <material>Gazebo/DarkGrey</material>
     </gazebo>
     <gazebo reference="right_wheel">
-        <material>Gazebo/BlackTransparent</material>
+        <material>Gazebo/DarkGrey</material>
     </gazebo>
     <gazebo reference="camera">

Commit message: .

File: my_robot/urdf/my_robot.xacro (robot description, xacro)
@@ -13,4 +13,5 @@
     </gazebo>
     <gazebo reference="camera">
+        <material>Gazebo/DarkGrey</material>
         <material>Gazebo/GreenTransparentOverlay</material>
     </gazebo>

Commit message: .

File: my_robot/urdf/my_robot.xacro (robot description, xacro)
@@ -13,6 +13,5 @@
     </gazebo>
     <gazebo reference="camera">
-        <material>Gazebo/DarkGrey</material>
-        <material>Gazebo/GreenTransparentOverlay</material>
+        <material>Gazebo/TurquoiseGlowOutline</material>
     </gazebo>
     <link name='chassis'>
