Commit message: .

File: my_robot/urdf/my_robot.xacro (robot description, xacro)
@@ -2,186 +2,187 @@
 <robot name="my_robot" xmlns:xacro="http://www.ros.org/wiki/xacro">
     <xacro:include filename="$(find my_robot)/urdf/my_robot.gazebo" />
-    <link name="robot_footprint"></link>
-    <!-- Model materials -->
-    <gazebo reference="chassis">
-        <material>Gazebo/Wood</material>
-    </gazebo>
-    <gazebo reference="left_wheel">
-        <material>Gazebo/DarkGrey</material>
-    </gazebo>
-    <gazebo reference="right_wheel">
-        <material>Gazebo/DarkGrey</material>
-    </gazebo>
-    <gazebo reference="camera">
-        <material>Gazebo/TurquoiseGlowOutline</material>
-    </gazebo>
-    <link name='chassis'>
-        <pose>0 0 0.1 0 0 0</pose>
-        <inertial>
-            <mass value="15.0" />
-            <origin xyz="0.0 0 0" rpy=" 0 0 0" />
-            <inertia
-                ixx="0.1" ixy="0" ixz="0"
-                iyy="0.1" iyz="0"
-                izz="0.1" />
-        </inertial>
-        <collision name='chassis_collision'>
-            <origin xyz="0 0 0" rpy=" 0 0 0" />
-            <geometry>
-                <box size=".4 .2 .1" />
-            </geometry>
-        </collision>
-        <visual name='chassis_visual'>
-            <origin xyz="0 0 0" rpy=" 0 0 0" />
-            <geometry>
-                <box size=".4 .2 .1" />
-            </geometry>
-        </visual>
-        <collision name='back_caster_collision'>
-            <origin xyz="-0.15 0 -0.05" rpy=" 0 0 0" />
-            <geometry>
-                <sphere radius="0.0499" />
-            </geometry>
-        </collision>
-        <visual name='back_caster_visual'>
-            <origin xyz="-0.15 0 -0.05" rpy=" 0 0 0" />
-            <geometry>
-                <sphere radius="0.05" />
-            </geometry>
-        </visual>
-        <collision name='front_caster_collision'>
-            <origin xyz="0.15 0 -0.05" rpy="0 0 0" />
-            <geometry>
-                <sphere radius="0.0499" />
-            </geometry>
-        </collision>
-        <visual name='front_caster_visual'>
-            <origin xyz="0.15 0 -0.05" rpy="0 0 0" />
-            <geometry>
-                <sphere radius="0.05" />
-            </geometry>
-        </visual>
+    <link name="robot_footprint">
+        <link name='chassis'>
+            <pose>0 0 0.1 0 0 0</pose>
+            <inertial>
+                <mass value="15.0" />
+                <origin xyz="0.0 0 0" rpy=" 0 0 0" />
+                <inertia
+                    ixx="0.1" ixy="0" ixz="0"
+                    iyy="0.1" iyz="0"
+                    izz="0.1" />
+            </inertial>
+            <collision name='chassis_collision'>
+                <origin xyz="0 0 0" rpy=" 0 0 0" />
+                <geometry>
+                    <box size=".4 .2 .1" />
+                </geometry>
+            </collision>
+            <visual name='chassis_visual'>
+                <origin xyz="0 0 0" rpy=" 0 0 0" />
+                <geometry>
+                    <box size=".4 .2 .1" />
+                </geometry>
+            </visual>
+            <collision name='back_caster_collision'>
+                <origin xyz="-0.15 0 -0.05" rpy=" 0 0 0" />
+                <geometry>
+                    <sphere radius="0.0499" />
+                </geometry>
+            </collision>
+            <visual name='back_caster_visual'>
+                <origin xyz="-0.15 0 -0.05" rpy=" 0 0 0" />
+                <geometry>
+                    <sphere radius="0.05" />
+                </geometry>
+            </visual>
+            <collision name='front_caster_collision'>
+                <origin xyz="0.15 0 -0.05" rpy="0 0 0" />
+                <geometry>
+                    <sphere radius="0.0499" />
+                </geometry>
+            </collision>
+            <visual name='front_caster_visual'>
+                <origin xyz="0.15 0 -0.05" rpy="0 0 0" />
+                <geometry>
+                    <sphere radius="0.05" />
+                </geometry>
+            </visual>
+        </link>
+        <joint name="robot_footprint_joint" type="fixed">
+            <origin xyz="0 0 0" rpy="0 0 0" />
+            <parent link="robot_footprint" />
+            <child link="chassis" />
+        </joint>
+        <link name='left_wheel'>
+            <inertial>
+                <mass value="5.0" />
+                <origin xyz="0.0 0 0" rpy="0 0 0" />
+                <inertia
+                    ixx="0.1" ixy="0" ixz="0"
+                    iyy="0.1" iyz="0"
+                    izz="0.1" />
+            </inertial>
+            <visual name='left_wheel_visual'>
+                <origin xyz="0 0 0" rpy="0 1.5707 1.5707" />
+                <geometry>
+                    <cylinder radius="0.1" length="0.05" />
+                </geometry>
+            </visual>
+            <collision name='left_wheel_collision'>
+                <origin xyz="0 0 0" rpy="0 1.5707 1.5707" />
+                <geometry>
+                    <cylinder radius="0.099" length="0.0499" />
+                </geometry>
+            </collision>
+        </link>
+        <joint type="continuous" name="left_wheel_hinge">
+            <origin xyz="0 0.15 0" rpy="0 0 0" />
+            <child link="left_wheel" />
+            <parent link="chassis" />
+            <axis xyz="0 1 0" rpy="0 0 0" />
+            <limit effort="10000" velocity="1000" />
+            <dynamics damping="1.0" friction="1.0" />
+        </joint>
+        <link name='right_wheel'>
+            <inertial>
+                <mass value="5.0" />
+                <origin xyz="0.0 0 0" rpy=" 0 0 0" />
+                <inertia
+                    ixx="0.1" ixy="0" ixz="0"
+                    iyy="0.1" iyz="0"
+                    izz="0.1" />
+            </inertial>
+            <visual name='right_wheel_visual'>
+                <origin xyz="0 0 0" rpy="0 1.5707 1.5707" />
+                <geometry>
+                    <cylinder radius="0.1" length="0.05" />
+                </geometry>
+            </visual>
+            <collision name='right_wheel_collision'>
+                <origin xyz="0 0 0" rpy="0 1.5707 1.5707" />
+                <geometry>
+                    <cylinder radius="0.099" length="0.0499" />
+                </geometry>
+            </collision>
+        </link>
+        <joint type="continuous" name="right_wheel_hinge">
+            <origin xyz="0 -0.15 0" rpy="0 0 0" />
+            <child link="right_wheel" />
+            <parent link="chassis" />
+            <axis xyz="0 1 0" rpy="0 0 0" />
+            <limit effort="10000" velocity="1000" />
+            <dynamics damping="1.0" friction="1.0" />
+        </joint>
+        <!-- Camera link -->
+        <link name="camera">
+            <origin xyz="0 0 0" rpy="0 0 0" />
+            <inertial>
+                <mass value="0.1" />
+                <origin xyz="0 0 0" rpy="0 0 0" />
+                <inertia ixx="1e-6" ixy="0" ixz="0" iyy="1e-6" iyz="0" izz="1e-6" />
+            </inertial>
+            <visual>
+                <origin xyz="0 0 0" rpy="0 0 0" />
+                <geometry>
+                    <box size="0.05 0.05 0.05" />
+                </geometry>
+                <material name="grey" />
+            </visual>
+            <collision>
+                <origin xyz="0 0 0" rpy="0 0 0" />
+                <geometry>
+                    <box size="0.05 0.05 0.05" />
+                </geometry>
+            </collision>
+        </link>
+        <!-- Camera joint -->
+        <joint name="camera_joint" type="fixed">
+            <parent link="chassis" />
+            <child link="camera" />
+            <origin xyz="0.2 0 0" rpy="0 0 0" />
+            <axis xyz="0 1 0" />
+        </joint>
+        <!-- Hokuyo LiDAR link -->
+        <link name="hokuyo">
+            <origin xyz="0 0 0" rpy="0 0 0" />
+            <inertial>
+                <mass value="1e-5" />
+                <origin xyz="0 0 0" rpy="0 0 0" />
+                <inertia ixx="1e-6" ixy="0" ixz="0" iyy="1e-6" iyz="0" izz="1e-6" />
+            </inertial>
+            <visual>
+                <origin xyz="0 0 0" rpy="0 0 0" />
+                <geometry>
+                    <mesh filename="package://my_robot/meshes/hokuyo.dae" />
+                </geometry>
+            </visual>
+            <collision>
+                <origin xyz="0 0 0" rpy="0 0 0" />
+                <geometry>
+                    <box size="0.1 0.1 0.1" />
+                </geometry>
+            </collision>
+        </link>
+        <!-- Hokuyo LiDAR joint -->
+        <joint name="hokuyo_joint" type="fixed">
+            <parent link="chassis" />
+            <child link="hokuyo" />
+            <origin xyz="0.15 0 0.1" rpy="0 0 0" />
+            <axis xyz="0 1 0" />
+        </joint>
+        <!-- Model materials -->
+        <gazebo reference="chassis">
+            <material>Gazebo/Wood</material>
+        </gazebo>
+        <gazebo reference="left_wheel">
+            <material>Gazebo/DarkGrey</material>
+        </gazebo>
+        <gazebo reference="right_wheel">
+            <material>Gazebo/DarkGrey</material>
+        </gazebo>
+        <gazebo reference="camera">
+            <material>Gazebo/TurquoiseGlowOutline</material>
+        </gazebo>
     </link>
-    <joint name="robot_footprint_joint" type="fixed">
-        <origin xyz="0 0 0" rpy="0 0 0" />
-        <parent link="robot_footprint" />
-        <child link="chassis" />
-    </joint>
-    <link name='left_wheel'>
-        <inertial>
-            <mass value="5.0" />
-            <origin xyz="0.0 0 0" rpy="0 0 0" />
-            <inertia
-                ixx="0.1" ixy="0" ixz="0"
-                iyy="0.1" iyz="0"
-                izz="0.1" />
-        </inertial>
-        <visual name='left_wheel_visual'>
-            <origin xyz="0 0 0" rpy="0 1.5707 1.5707" />
-            <geometry>
-                <cylinder radius="0.1" length="0.05" />
-            </geometry>
-        </visual>
-        <collision name='left_wheel_collision'>
-            <origin xyz="0 0 0" rpy="0 1.5707 1.5707" />
-            <geometry>
-                <cylinder radius="0.099" length="0.0499" />
-            </geometry>
-        </collision>
-    </link>
-    <joint type="continuous" name="left_wheel_hinge">
-        <origin xyz="0 0.15 0" rpy="0 0 0" />
-        <child link="left_wheel" />
-        <parent link="chassis" />
-        <axis xyz="0 1 0" rpy="0 0 0" />
-        <limit effort="10000" velocity="1000" />
-        <dynamics damping="1.0" friction="1.0" />
-    </joint>
-    <link name='right_wheel'>
-        <inertial>
-            <mass value="5.0" />
-            <origin xyz="0.0 0 0" rpy=" 0 0 0" />
-            <inertia
-                ixx="0.1" ixy="0" ixz="0"
-                iyy="0.1" iyz="0"
-                izz="0.1" />
-        </inertial>
-        <visual name='right_wheel_visual'>
-            <origin xyz="0 0 0" rpy="0 1.5707 1.5707" />
-            <geometry>
-                <cylinder radius="0.1" length="0.05" />
-            </geometry>
-        </visual>
-        <collision name='right_wheel_collision'>
-            <origin xyz="0 0 0" rpy="0 1.5707 1.5707" />
-            <geometry>
-                <cylinder radius="0.099" length="0.0499" />
-            </geometry>
-        </collision>
-    </link>
-    <joint type="continuous" name="right_wheel_hinge">
-        <origin xyz="0 -0.15 0" rpy="0 0 0" />
-        <child link="right_wheel" />
-        <parent link="chassis" />
-        <axis xyz="0 1 0" rpy="0 0 0" />
-        <limit effort="10000" velocity="1000" />
-        <dynamics damping="1.0" friction="1.0" />
-    </joint>
-    <!-- Camera link -->
-    <link name="camera">
-        <origin xyz="0 0 0" rpy="0 0 0" />
-        <inertial>
-            <mass value="0.1" />
-            <origin xyz="0 0 0" rpy="0 0 0" />
-            <inertia ixx="1e-6" ixy="0" ixz="0" iyy="1e-6" iyz="0" izz="1e-6" />
-        </inertial>
-        <visual>
-            <origin xyz="0 0 0" rpy="0 0 0" />
-            <geometry>
-                <box size="0.05 0.05 0.05" />
-            </geometry>
-            <material name="grey" />
-        </visual>
-        <collision>
-            <origin xyz="0 0 0" rpy="0 0 0" />
-            <geometry>
-                <box size="0.05 0.05 0.05" />
-            </geometry>
-        </collision>
-    </link>
-    <!-- Camera joint -->
-    <joint name="camera_joint" type="fixed">
-        <parent link="chassis" />
-        <child link="camera" />
-        <origin xyz="0.2 0 0" rpy="0 0 0" />
-        <axis xyz="0 1 0" />
-    </joint>
-    <!-- Hokuyo LiDAR link -->
-    <link name="hokuyo">
-        <origin xyz="0 0 0" rpy="0 0 0" />
-        <inertial>
-            <mass value="1e-5" />
-            <origin xyz="0 0 0" rpy="0 0 0" />
-            <inertia ixx="1e-6" ixy="0" ixz="0" iyy="1e-6" iyz="0" izz="1e-6" />
-        </inertial>
-        <visual>
-            <origin xyz="0 0 0" rpy="0 0 0" />
-            <geometry>
-                <mesh filename="package://my_robot/meshes/hokuyo.dae" />
-            </geometry>
-        </visual>
-        <collision>
-            <origin xyz="0 0 0" rpy="0 0 0" />
-            <geometry>
-                <box size="0.1 0.1 0.1" />
-            </geometry>
-        </collision>
-    </link>
-    <!-- Hokuyo LiDAR joint -->
-    <joint name="hokuyo_joint" type="fixed">
-        <parent link="chassis" />
-        <child link="hokuyo" />
-        <origin xyz="0.15 0 0.1" rpy="0 0 0" />
-        <axis xyz="0 1 0" />
-    </joint>
 </robot>
