Commit message: .

File: my_robot/urdf/my_robot.xacro (robot description, xacro)
@@ -126,5 +126,5 @@
     </inertial>
     <visual>
-      <origin xyz="0.15 0 0" rpy="0 0 0" />
+      <origin xyz="0.1 0 0" rpy="0 0 0" />
       <geometry>
         <box size="0.05 0.05 0.05" />
@@ -133,5 +133,5 @@
     </visual>
     <collision>
-      <origin xyz="0.15 0 0" rpy="0 0 0" />
+      <origin xyz="0.1 0 0" rpy="0 0 0" />
       <geometry>
         <box size="0.05 0.05 0.05" />
@@ -143,5 +143,5 @@
     <parent link="chassis" />
     <child link="camera" />
-    <origin xyz="0.2 0 0" rpy="0 0 0" />
+    <origin xyz="0.1 0 0" rpy="0 0 0" />
     <axis xyz="0 1 0" />
   </joint>

Commit message: .

File: my_robot/urdf/my_robot.xacro (robot description, xacro)
@@ -126,5 +126,5 @@
     </inertial>
     <visual>
-      <origin xyz="0.1 0 0" rpy="0 0 0" />
+      <origin xyz="0 0 0" rpy="0 0 0" />
       <geometry>
         <box size="0.05 0.05 0.05" />
@@ -133,5 +133,5 @@
     </visual>
     <collision>
-      <origin xyz="0.1 0 0" rpy="0 0 0" />
+      <origin xyz="0 0 0" rpy="0 0 0" />
       <geometry>
         <box size="0.05 0.05 0.05" />
@@ -143,5 +143,5 @@
     <parent link="chassis" />
     <child link="camera" />
-    <origin xyz="0.1 0 0" rpy="0 0 0" />
+    <origin xyz="0.2 0 0" rpy="0 0 0" />
     <axis xyz="0 1 0" />
   </joint>

Commit message: .

File: my_robot/urdf/my_robot.xacro (robot description, xacro)
@@ -151,9 +151,9 @@
     <inertial>
       <mass value="1e-5" />
-      <origin xyz="0 0 0.05" rpy="0 0 0" />
+      <origin xyz="0 0 0" rpy="0 0 0" />
       <inertia ixx="1e-6" ixy="0" ixz="0" iyy="1e-6" iyz="0" izz="1e-6" />
     </inertial>
     <visual>
-      <origin xyz="0.05 0 0.03" rpy="0 0 0" />
+      <origin xyz="0 0 0" rpy="0 0 0" />
       <geometry>
         <mesh filename="package://my_robot/meshes/hokuyo.dae" />
@@ -161,5 +161,5 @@
     </visual>
     <collision>
-      <origin xyz="0.05 0 0.03" rpy="0 0 0" />
+      <origin xyz="0 0 0" rpy="0 0 0" />
       <geometry>
         <box size="0.1 0.1 0.1" />

Commit message: change camera link material grey to Gazebo/Grey

File: my_robot/urdf/my_robot.xacro (robot description, xacro)
@@ -129,5 +129,6 @@
         <box size="0.05 0.05 0.05" />
       </geometry>
-      <material name="grey" />
+      <!-- <material name="grey" /> -->
+      <material name="Gazebo/Grey" />
     </visual>
     <collision>

Commit message: .

File: my_robot/urdf/my_robot.xacro (robot description, xacro)
@@ -130,5 +130,4 @@
       </geometry>
       <!-- <material name="grey" /> -->
-      <material name="Gazebo/Grey" />
     </visual>
     <collision>

Commit message: change robot car wheels

File: my_robot/urdf/my_robot.xacro (robot description, xacro)
@@ -1,6 +1,6 @@
 <?xml version='1.0'?>
 <robot name="my_robot" xmlns:xacro="http://www.ros.org/wiki/xacro">
-  <!--Import gazebo elements-->
   <xacro:include filename="$(find my_robot)/urdf/my_robot.gazebo" />
+  <!-- Import gazebo elements -->
   <link name="robot_footprint" />
   <link name='chassis'>
@@ -56,4 +56,5 @@
     <child link="chassis" />
   </joint>
+  <!-- Left Wheel -->
   <link name='left_wheel'>
     <inertial>
@@ -62,11 +63,10 @@
       <inertia
         ixx="0.1" ixy="0" ixz="0"
-        iyy="0.1" iyz="0"
-        izz="0.1" />
+        iyy="0.1" iyz="0" izz="0.1" />
     </inertial>
     <visual name='left_wheel_visual'>
       <origin xyz="0 0 0" rpy="0 1.5707 1.5707" />
       <geometry>
-        <cylinder radius="0.1" length="0.05" />
+        <cylinder radius="0.101" length="0.05" />
       </geometry>
     </visual>
@@ -74,8 +74,9 @@
       <origin xyz="0 0 0" rpy="0 1.5707 1.5707" />
       <geometry>
-        <cylinder radius="0.099" length="0.0499" />
+        <cylinder radius="0.101" length="0.05" />
       </geometry>
     </collision>
   </link>
+  <!-- Left Wheel Hinge -->
   <joint type="continuous" name="left_wheel_hinge">
     <origin xyz="0 0.15 0" rpy="0 0 0" />
@@ -98,5 +99,5 @@
       <origin xyz="0 0 0" rpy="0 1.5707 1.5707" />
       <geometry>
-        <cylinder radius="0.1" length="0.05" />
+        <cylinder radius="0.101" length="0.05" />
       </geometry>
     </visual>
@@ -104,5 +105,5 @@
       <origin xyz="0 0 0" rpy="0 1.5707 1.5707" />
       <geometry>
-        <cylinder radius="0.099" length="0.0499" />
+        <cylinder radius="0.101" length="0.05" />
       </geometry>
     </collision>
@@ -120,5 +121,5 @@
     <origin xyz="0 0 0" rpy="0 0 0" />
     <inertial>
-      <mass value="0.1" />
+      <mass value="1e-5" />
       <origin xyz="0 0 0" rpy="0 0 0" />
       <inertia ixx="1e-6" ixy="0" ixz="0" iyy="1e-6" iyz="0" izz="1e-6" />
